File: OshTeledongle.kicad_pcb (KiCad board)
At the start: 4 copper layers, 35 x 84 mm, 47 parts, among them J1 SMA_Edgelaunch, J2 Conn_ARM_SWD_TagConnect_TC203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, J3 Conn_01x02, J4 USB_C_Receptacle_USB2.0_16P, J5 Conn_01x02, SW1 SW_Push_SPDT, U17 MCP73831-2-OT, U18 AP131-33, U2 WE-TVS-82400102, U3 STM32F042C4Tx, U4 RN4678-V/RM113, Y2 ECS-320-8-33Q-JES-TR

Commit message: v1.1 release, fixed a spi pin disconnected, should be good for mass prod now
Connections:
- U5 pad 8: /MOSI3 -> /MOSI2
Routing:
- net /MOSI2: track 0.00 -> 38.6 mm, vias 0 -> 2
Other:
- board text added: "RE-leBT v1.1"
- board text removed: "RE-leBT v1.0"
