File: OshTeledongle.kicad_sch (KiCad schematic)
At the start: 47 parts, among them J1 USB_C_Receptacle_USB2.0_16P, J2 Conn_ARM_SWD_TagConnect_TC203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, J3 SMA_Edgelaunch, U1 AP2112K-3.3, U2 WE-TVS-82400102, U3 STM32F042C4Tx, U8 CC1200, Y1 ABM8W-40.0000MHZ

Commit message: v1.0 done
Parts:
- removed J1: USB_C_Receptacle_USB2.0_16P, Connector_USB:USB_C_Receptacle_G-Switch_GT-USB-7010ASV, symbol Connector:USB_C_Receptacle_USB2.0_16P
- added C43: 1uF, Capacitor_SMD:C_0402_1005Metric, symbol Device:C
- added C44, C47: 0.1uF, Capacitor_SMD:C_0402_1005Metric, symbol Device:C
- added C45, C46: 8pF, Capacitor_SMD:C_0402_1005Metric, symbol Device:C
- added D1: RED, LED_SMD:LED_0603_1608Metric, symbol Device:LED
- added D2: BLUE, LED_SMD:LED_0603_1608Metric, symbol Device:LED
- added FB1: FerriteBead_Small, Inductor_SMD:L_0402_1005Metric, symbol Device:FerriteBead_Small
- added H1, H2: MountingHole_Pad, MountingHole:MountingHole_3.2mm_M3_DIN965_Pad, symbol Mechanical:MountingHole_Pad
- added J4: USB_C_Receptacle_USB2.0_16P, Connector_USB:USB_C_Receptacle_GCT_USB4105-xx-A_16P_TopMnt_Horizontal, symbol Connector:USB_C_Receptacle_USB2.0_16P
- added R11, R13: 1k, Resistor_SMD:R_0402_1005Metric, symbol Device:R
- added R3: 56k, Resistor_SMD:R_0402_1005Metric, symbol Device:R
- added U4: RN4678-V/RM113, FCU2025Lib:RN4678_MCH, symbol FCU2025:RN4678-V_RM113
- added Y2: ECS-320-8-33Q-JES-TR, Crystal:Crystal_SMD_Abracon_ABM8G-4Pin_3.2x2.5mm, symbol Device:Crystal_GND24_Small
Connections:
- net +3V3: now also U3.1 (VBAT), U3.24 (VDD), U3.36 (VDDIO2), U3.48 (VDD), C47.1, FB1.1, U4.4 (BAT_IN)
- net CS_RADIO: now also U3.22 (PB11)
- net GND: now also C43.1, C44.1, C45.1, C46.1, C47.2, D1.1 (K), D2.1 (K), H1.1, H2.1, J4.A1 (GND), J4.A12 (GND), J4.B1 (GND), J4.B12 (GND), J4.S1 (SHIELD), R3.1, U4.1 (GND), U4.2 (GND), U4.3 (GND), U4.31 (GND), U4.32 (GND), U4.33 (GND), Y2.2, Y2.4
- net MISO2: now also U3.16 (PA6)
- net MOSI2: now also U3.17 (PA7)
- net RADIO_INT: now also U3.21 (PB10)
- net SCK2: now also U3.15 (PA5)
- net USB_D+: now also U3.33 (PA12)
- net USB_D-: now also U3.32 (PA11)
- net VBUS: now also J4.A4 (VBUS), J4.A9 (VBUS), J4.B4 (VBUS), J4.B9 (VBUS)
- net at R9.1: now also J4.A7 (D-), J4.B7 (D-)
- net at R1.1: now also J4.A5 (CC1)
- net at R2.1: now also J4.B5 (CC2)
- net at R10.1: now also J4.A6 (D+), J4.B6 (D+)
- net CTS2: now reaches U3.10 (PA0)
- net CTS2: now also U4.17 (P0_0/RTS)
- net RTS2: now reaches U3.11 (PA1)
- net RTS2: now also U4.15 (P1_7/CTS)
- net TX2: now reaches U3.12 (PA2)
- net TX2: now also U4.22 (RXD)
- net RX2: now reaches U3.13 (PA3)
- net RX2: now also U4.23 (TXD)
- net VDIV: now reaches U3.14 (PA4)
- net at U3.18 (PB0): now also R11.2
- net BT_P0_4: now reaches U3.2 (PC13)
- net BT_P0_4: now also U4.11 (P0_4)
- net BT_P3_1: now reaches U3.20 (PB2)
- net BT_P3_1: now also U4.24 (P3_1)
- net BT_P3_7: now reaches U3.25 (PB12)
- net BT_P3_7: now also U4.29 (P3_7)
- net BT_P3_6: now reaches U3.26 (PB13)
- net BT_P3_6: now also U4.28 (P3_6)
- net BT_P3_4: now reaches U3.27 (PB14)
- net BT_P3_4: now also U4.27 (P3_4)
- net BT_P3_3: now reaches U3.28 (PB15)
- net BT_P3_3: now also U4.26 (P3_3)
- net BT_P3_2: now reaches U3.29 (PA8)
- net BT_P3_2: now also U4.25 (P3_2)
- net BT_SW_BTN: now reaches U3.3 (PC14)
- net BT_SW_BTN: now also U4.5 (SW_BTN)
- net BT_P2_4: now reaches U3.31 (PA10)
- net BT_P2_4: now also U4.19 (P2_4)
- net BT_NRST: now reaches U3.38 (PA15)
- net BT_NRST: now also R3.2, U4.21 (*RST_N)
- net BT_P2_0: now reaches U3.39 (PB3)
- net BT_P2_0: now also U4.18 (P2_0)
- net at U3.4 (PC15): now also R13.2
- net BT_P0_5: now reaches U3.41 (PB5)
- net BT_P0_5: now also U4.16 (P0_5)
- net BT_P1_5: now reaches U3.42 (PB6)
- net BT_P1_5: now also U4.12 (P1_5)
- net BT_P1_2: now reaches U3.43 (PB7)
- net BT_P1_2: now also U4.13 (P1_2)
- net BT_WAKE: now reaches U3.46 (PB9)
- net BT_WAKE: now also U4.9 (WAKEUP)
- net PF0: now reaches U3.5 (PF0)
- net PF0: now also C46.2, Y2.1
- net PF1: now reaches U3.6 (PF1)
- net PF1: now also C45.2, Y2.3
- net at U3.9 (VDDA): now also C43.2, C44.2, FB1.2
- new net: D1.2 (A), R11.1
- new net: U4.6 (LDO33_O), U4.7 (VDD_IO)
- new net: D2.2 (A), R13.1
- no-connect marks 1 -> 10
Other:
- moved on the sheet: C1, C2, U1, U3

Commit message: v1.0 sent to fab
Parts:
- removed C11, C12, C14, C15, C28, C29, C30, C32, C34: 47nF, Capacitor_SMD:C_0402_1005Metric, symbol Device:C
- removed C13: 0.22uF, Capacitor_SMD:C_0402_1005Metric, symbol Device:C
- removed C25, C26: 10pF, Capacitor_SMD:C_0402_1005Metric, symbol Device:C
- removed C27: 1.8nF, Capacitor_SMD:C_0402_1005Metric, symbol Device:C
- removed C31: 56pF, Capacitor_SMD:C_0402_1005Metric, symbol Device:C
- removed C33, C35: 10nF, Capacitor_SMD:C_0402_1005Metric, symbol Device:C
- removed C36: 100pF, Capacitor_SMD:C_0402_1005Metric, symbol Device:C
- removed C37, C38, C39: 5.1pF, Capacitor_SMD:C_0402_1005Metric, symbol Device:C
- removed C40: 39pF, Capacitor_SMD:C_0402_1005Metric, symbol Device:C
- removed C41: 2.2pF, Capacitor_SMD:C_0402_1005Metric, symbol Device:C
- removed C42: 6.2pF, Capacitor_SMD:C_0402_1005Metric, symbol Device:C
- removed J3: SMA_Edgelaunch, Connector_Coaxial:SMA_Amphenol_132289_EdgeMount, symbol Connector:Conn_Coaxial
- removed L1, L2: LQG15HS56NJ02D, Inductor_SMD:L_0402_1005Metric, symbol Device:L_Small
- removed L3, L4: LQG15HZ27NJ02D, Inductor_SMD:L_0402_1005Metric, symbol Device:L_Small
- removed L5, L6: LQG15HS15NJ02D, Inductor_SMD:L_0402_1005Metric, symbol Device:L_Small
- removed L7: MLG1005S43NJTD25, Inductor_SMD:L_0402_1005Metric, symbol Device:L_Small
- removed L8: LQG15HS22NG02D, Inductor_SMD:L_0402_1005Metric, symbol Device:L_Small
- removed R12: 56k, Resistor_SMD:R_0402_1005Metric, symbol Device:R
- removed R48: 18, Resistor_SMD:R_0402_1005Metric, symbol Device:R
- removed U1: AP2112K-3.3, Package_TO_SOT_SMD:SOT-23-5, symbol Regulator_Linear:AP2112K-3.3
- removed U8: CC1200, Package_DFN_QFN:QFN-32-1EP_5x5mm_P0.5mm_EP3.45x3.45mm, symbol RF:CC1200
- removed Y1: ABM8W-40.0000MHZ, Crystal:Crystal_SMD_Abracon_ABM8G-4Pin_3.2x2.5mm, symbol Device:Crystal_GND24_Small
- added C20, C21: 4.7uF, Capacitor_SMD:C_0402_1005Metric, symbol Device:C
- added C24: 1uF, Capacitor_SMD:C_0402_1005Metric, symbol Device:C
- added C3: 100nF, Capacitor_SMD:C_0402_1005Metric, symbol Device:C
- added C4: 10nF, Capacitor_SMD:C_0402_1005Metric, symbol Device:C
- added D3, D4: LED, LED_SMD:LED_0603_1608Metric, symbol Device:LED
- added H3: MountingHole_Pad, MountingHole:MountingHole_3.2mm_M3_DIN965_Pad, symbol Mechanical:MountingHole_Pad
- added J1: SMA_Edgelaunch, Connector_Coaxial:SMA_Amphenol_132289_EdgeMount, symbol Connector:Conn_Coaxial
- added J3: Conn_01x02, Connector_JST:JST_PH_S2B-PH-K_1x02_P2.00mm_Horizontal, symbol Connector_Generic:Conn_01x02
- added J5: Conn_01x02, Connector_PinHeader_2.54mm:PinHeader_1x02_P2.54mm_Vertical, symbol Connector_Generic:Conn_01x02
- added R37: 2.49k, Resistor_SMD:R_0402_1005Metric, symbol Device:R
- added R4, R5: 1k, Resistor_SMD:R_0402_1005Metric, symbol Device:R
- added R6: 10k, Resistor_SMD:R_0402_1005Metric, symbol Device:R
- added R7: 5.1k, Resistor_SMD:R_0402_1005Metric, symbol Device:R
- added SW1: SW_Push_SPDT, Button_Switch_THT:SW_E-Switch_EG1224_SPDT_Angled, symbol Switch:SW_Push_SPDT
- added U17: MCP73831-2-OT, Package_TO_SOT_SMD:SOT-23-5, symbol Battery_Management:MCP73831-2-OT
- added U18: AP131-33, Package_TO_SOT_SMD:SOT-23-5, symbol Regulator_Linear:TC2185-3.3VxCTTR
- added U5: ~, FCU2025Lib:N511CS, symbol FCU2025:N511CS-B_CC1200
- C2: value 1uF -> 100nF
Connections:
- net +3V3: now also C24.2, C3.2, U18.5 (VOUT), U5.13 (VCC), U5.6 (VTC)
- net CS_RADIO: now also U5.12 (CS)
- net GND: now also C20.1, C21.1, C24.1, C3.1, C4.1, H3.1, J1.2 (Ext), J3.2 (Pin_2), J5.2 (Pin_2), R37.1, R5.1, R6.1, U17.2 (V_{SS}), U18.2 (GND), U5.14 (GND), U5.2 (GND), U5.3 (GND)
- net MISO2: now also U5.10 (MISO)
- net NRST: now also U5.5 (NRST)
- net RADIO_INT: now also U5.7 (GPIO2)
- net RADIO_MARC_ISR: now also U5.4 (GPIO3)
- net SCK2: now also U5.9 (SCK)
- net VBUS: now also C20.2, R4.2, U17.4 (V_{DD}); no longer C1.2
- net at U3.30 (PA9): now also J5.1 (Pin_1)
- net VDIV renamed V_BATT
- net V_BATT: now also R6.2, R7.1
- new net: C4.2, U18.4 (BP)
- new net: C1.2, SW1.3 (C), U18.1 (VIN), U18.3 (ON/~{OFF})
- new net: D3.2 (A), D4.1 (K), U17.1 (STAT)
- new net: D4.2 (A), R4.1
- new net: D3.1 (K), R5.2
- new net: J1.1 (In), U5.1 (RF)
- new net: R37.2, U17.5 (PROG)
- new net MOSI3: U5.8 (MOSI)
- new net V_CHARGE: C21.2, J3.1 (Pin_1), R7.2, SW1.2 (B), U17.3 (V_{BAT})
- no-connect marks 10 -> 9
Other:
- moved on the sheet: C43, C44, C45, C46, C47, D1, D2, FB1, H1, H2, R11, R13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
