File: OshTeledongle.kicad_sch (KiCad schematic)
At the start: 45 parts, among them J1 SMA_Edgelaunch, J2 Conn_ARM_SWD_TagConnect_TC203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, J3 Conn_01x02, J4 USB_C_Receptacle_USB2.0_16P, J5 Conn_01x02, SW1 SW_Push_SPDT, U17 MCP73831-2-OT, U18 AP131-33, U2 WE-TVS-82400102, U3 STM32F042C4Tx, U4 RN4678-V/RM113, Y2 ECS-320-8-33Q-JES-TR

Commit message: v1.1 release, fixed a spi pin disconnected, should be good for mass prod now
Connections:
- net MOSI3 is gone; now on net MOSI2: U5.8 (MOSI)
Changed lines of the file:
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@@
 	(generator_version "9.0")
 	(paper "A4")
+	(title_block
+		(rev "1.1")
+	)
 	(text "RADIO"
 		(exclude_from_sim no)
@@
 		)
 	)
-	(label "MOSI3"
+	(label "MOSI2"
 		(at 204.47 45.72 0)
 		(effects
